Commit message: fix 1.0

File: competition/erc_v1_0_0/src/erc_description/urdf/tiago_pro.urdf (robot description, URDF)
Before this commit: robot tiago_pro, 84 links, 83 joints
Links:
- link gripper_left_fingertip_left_link: geometry collision box size=0.04 0.07 0.034; visual mesh filename=package://pal_pro_gripper_description/meshes/fingertip.stl
- link gripper_left_fingertip_right_link: geometry collision box size=0.04 0.07 0.034; visual mesh filename=package://pal_pro_gripper_description/meshes/fingertip.stl

Commit message: fix 2.0 the gripper

File: competition/erc_v1_0_0/src/erc_description/urdf/tiago_pro.urdf (robot description, URDF)
Before this commit: robot tiago_pro, 84 links, 83 joints
Links:
- link gripper_left_fingertip_left_link: geometry collision mesh filename=package://pal_pro_gripper_description/meshes/fingertip.stl; visual mesh filename=package://pal_pro_gripper_description/meshes/fingertip.stl
- link gripper_left_fingertip_right_link: geometry collision mesh filename=package://pal_pro_gripper_description/meshes/fingertip.stl; visual mesh filename=package://pal_pro_gripper_description/meshes/fingertip.stl
